Commit message: [Visual] - Phase 6: OBJ mesh + 4-wheel robot visual upgrade
- Replace all primitive visuals (box/cylinder/STL) with Blender OBJ meshes
  for baselink, 4 wheels, lidar, camera
- Add texture support: MTL files with map_Kd PNG textures (logo_decal, vkuv)
- Convert 2-wheel+caster to 4-wheel drive (front/back left/right)
- Update wheel_link macro: add vis_x/y/z/rpy params for per-wheel mesh alignment
- Remove Gazebo/DarkGrey material override to allow OBJ/MTL textures to render
- Set GZ_SIM_RESOURCE_PATH to include obj/ texture dir for OGRE2 texture loading
- Update DiffDrive plugin to drive all 4 wheel joints
- Update xacro properties: chassis 0.8x0.8x0.6m, wheel_radius/width 0.08m
- Add phase_06 prompt doc and update HOW_TO_NAVIGATE

Made-with: Cursor

File: src/anhc_description/urdf/anhc_bot.urdf.xacro (robot description, xacro)
@@ -38,6 +38,8 @@
     <origin xyz="0 0 0" rpy="0 0 0"/>
   </joint>
-  <!-- Primitive wheel model (no external OBJ dependency). -->
-  <xacro:macro name="wheel_link" params="name x y">
+  <!-- mesh_file: OBJ filename under meshes/anhc_botrl/visual/obj/ -->
+  <!-- vis_x/y/z: visual origin offset in link frame (forward / left-right / up-down).       -->
+  <!-- vis_rpy:   visual rotation; default +90° roll. Use -1.5708 0 0 to flip inner/outer.  -->
+  <xacro:macro name="wheel_link" params="name x y mesh_file vis_x vis_y vis_z vis_rpy:='1.5708 0 0'">
     <link name="${name}">
       <inertial>
@@ -46,12 +48,11 @@
         <inertia ixx="0.0022" ixy="0.0" ixz="0.0" iyy="0.0040" iyz="0.0" izz="0.0022"/>
       </inertial>
+      <!-- OBJ from Blender in metres; scale = 1 1 1. MTL auto-loaded by matching base name. -->
       <visual>
-        <origin xyz="0 0 0" rpy="1.5708 0 0"/>
+        <origin xyz="${vis_x} ${vis_y} ${vis_z}" rpy="${vis_rpy}"/>
         <geometry>
-          <cylinder radius="${wheel_radius}" length="${wheel_width}"/>
+          <mesh filename="package://anhc_description/meshes/anhc_botrl/visual/obj/${mesh_file}"
+                scale="1 1 1"/>
         </geometry>
-        <material name="wheel_dark_gray">
-          <color rgba="0.10 0.10 0.10 1.0"/>
-        </material>
       </visual>
       <collision>
@@ -72,9 +73,12 @@
   </xacro:macro>
   <!-- Front wheels (powered, drive wheels) -->
-  <xacro:wheel_link name="front_left_wheel"  x="${wheel_x}"                    y="${wheel_y}"/>
-  <xacro:wheel_link name="front_right_wheel" x="${wheel_x}"                    y="-${wheel_y}"/>
+  <xacro:wheel_link name="front_left_wheel"  x="${wheel_x}"                    y="${wheel_y}"  mesh_file="front_left_wheel.obj"  vis_x="-0.0085" vis_y="0.0781"  vis_z="-0.0921"/>
+  <!-- vis_y/z computed for exact mirror symmetry with front_left (center_y=-0.05, center_z=-0.02) -->
+  <xacro:wheel_link name="front_right_wheel" x="${wheel_x}"                    y="-${wheel_y}" mesh_file="back_right_wheel.obj"  vis_x="-0.22" vis_y="0.1964"  vis_z="0.0542"  vis_rpy="-1.5708 0 0"/>
   <!-- Rear wheels — same joint type (continuous), driven passively via physics -->
-  <xacro:wheel_link name="back_left_wheel"   x="-${chassis_length/2.0 - 0.05}" y="${wheel_y}"/>
-  <xacro:wheel_link name="back_right_wheel"  x="-${chassis_length/2.0 - 0.05}" y="-${wheel_y}"/>
+  <!-- back_left: vis_x +0.04 (≈ half wheel width forward) -->
+  <xacro:wheel_link name="back_left_wheel"   x="-${chassis_length/2.0 - 0.05}" y="${wheel_y}"  mesh_file="back_left_wheel.obj"   vis_x="0.12"    vis_y="0.0655"  vis_z="-0.0986"/>
+  <!-- vis_y/z computed for exact mirror symmetry with back_left (center_y=-0.05, center_z=-0.021) -->
+  <xacro:wheel_link name="back_right_wheel"  x="-${chassis_length/2.0 - 0.05}" y="-${wheel_y}" mesh_file="front_right_wheel.obj" vis_x="0.50"    vis_y="0.0234"  vis_z="-0.0782"/>
   <link name="lidar_link">
     <inertial>
