Commit message: [fixbug] - fix Teleop

File: src/anhc_description/urdf/anhc_bot.gazebo.xacro (robot description, xacro)
@@ -98,7 +98,9 @@
       <max_linear_acceleration>0.8</max_linear_acceleration>
       <max_angular_acceleration>1.8</max_angular_acceleration>
-      <min_linear_velocity>-0.2</min_linear_velocity>
-      <cmd_vel_timeout>0.35</cmd_vel_timeout>
-      <topic>/cmd_vel</topic>
+      <!-- Symmetric limits; gz-sim8 DiffDrive ignores cmd_vel_timeout (not in plugin). -->
+      <min_linear_velocity>-0.35</min_linear_velocity>
+      <min_angular_velocity>-0.9</min_angular_velocity>
+      <!-- Omit <topic>: DiffDrive defaults to /model/<model_name>/cmd_vel (Harmonic/Garden).
+           A bare /cmd_vel + ros_gz_bridge often does not reach the plugin transport scope. -->
       <odom_topic>/odom</odom_topic>
       <tf_topic>/tf</tf_topic>

File: src/anhc_description/urdf/anhc_bot.urdf.xacro (robot description, xacro)
@@ -89,10 +89,5 @@
         </material>
       </visual>
-      <collision>
-        <origin xyz="0 0 0" rpy="0 0 0"/>
-        <geometry>
-          <sphere radius="0.04"/>
-        </geometry>
-      </collision>
+      <!-- No collision: passive casters + Gazebo contact solver often inject yaw torque. -->
     </link>
     <joint name="${name}_joint" type="fixed">
@@ -115,8 +110,5 @@
       <material name="blue"><color rgba="0.2 0.2 0.9 1.0"/></material>
     </visual>
-    <collision>
-      <origin xyz="0 0 0" rpy="0 0 0"/>
-      <geometry><cylinder radius="0.04" length="0.05"/></geometry>
-    </collision>
+    <!-- No collision: avoid spurious contacts with world mesh; lidar is not physical. -->
   </link>
   <joint name="lidar_joint" type="fixed">

Commit message: [Visual] - Phase 6: OBJ mesh + 4-wheel robot visual upgrade
- Replace all primitive visuals (box/cylinder/STL) with Blender OBJ meshes
  for baselink, 4 wheels, lidar, camera
- Add texture support: MTL files with map_Kd PNG textures (logo_decal, vkuv)
- Convert 2-wheel+caster to 4-wheel drive (front/back left/right)
- Update wheel_link macro: add vis_x/y/z/rpy params for per-wheel mesh alignment
- Remove Gazebo/DarkGrey material override to allow OBJ/MTL textures to render
- Set GZ_SIM_RESOURCE_PATH to include obj/ texture dir for OGRE2 texture loading
- Update DiffDrive plugin to drive all 4 wheel joints
- Update xacro properties: chassis 0.8x0.8x0.6m, wheel_radius/width 0.08m
- Add phase_06 prompt doc and update HOW_TO_NAVIGATE

Made-with: Cursor

File: src/anhc_description/urdf/anhc_bot.gazebo.xacro (robot description, xacro)
@@ -1,19 +1,8 @@
 <?xml version="1.0"?>
 <robot xmlns:xacro="http://www.ros.org/wiki/xacro">
-  <gazebo reference="base_link">
-    <material>Gazebo/DarkGrey</material>
-  </gazebo>
-  <gazebo reference="left_wheel">
-    <mu1>1.2</mu1>
-    <mu2>1.2</mu2>
-    <kp>100000.0</kp>
-    <kd>10.0</kd>
-  </gazebo>
-  <gazebo reference="right_wheel">
-    <mu1>1.2</mu1>
-    <mu2>1.2</mu2>
-    <kp>100000.0</kp>
-    <kd>10.0</kd>
-  </gazebo>
+  <gazebo reference="front_left_wheel">  <mu1>1.2</mu1><mu2>1.2</mu2><kp>100000.0</kp><kd>10.0</kd> </gazebo>
+  <gazebo reference="front_right_wheel"> <mu1>1.2</mu1><mu2>1.2</mu2><kp>100000.0</kp><kd>10.0</kd> </gazebo>
+  <gazebo reference="back_left_wheel">   <mu1>1.2</mu1><mu2>1.2</mu2><kp>100000.0</kp><kd>10.0</kd> </gazebo>
+  <gazebo reference="back_right_wheel">  <mu1>1.2</mu1><mu2>1.2</mu2><kp>100000.0</kp><kd>10.0</kd> </gazebo>
   <gazebo reference="lidar_link">
     <sensor name="anhc_lidar" type="gpu_lidar">
@@ -90,6 +79,9 @@
   <gazebo>
     <plugin filename="gz-sim-diff-drive-system" name="gz::sim::systems::DiffDrive">
-      <left_joint>left_wheel_joint</left_joint>
-      <right_joint>right_wheel_joint</right_joint>
+      <!-- 4WD: both left wheels share the same velocity command, same for right -->
+      <left_joint>front_left_wheel_joint</left_joint>
+      <left_joint>back_left_wheel_joint</left_joint>
+      <right_joint>front_right_wheel_joint</right_joint>
+      <right_joint>back_right_wheel_joint</right_joint>
       <wheel_separation>0.42</wheel_separation>
       <wheel_radius>0.08</wheel_radius>

File: src/anhc_description/urdf/anhc_bot.urdf.xacro (robot description, xacro)
@@ -1,14 +1,13 @@
 <?xml version="1.0"?>
 <robot xmlns:xacro="http://www.ros.org/wiki/xacro" name="anhc_bot">
-  <xacro:property name="chassis_length" value="0.5"/>
-  <xacro:property name="chassis_width" value="0.4"/>
-  <xacro:property name="chassis_height" value="0.25"/>
-  <xacro:property name="wheel_radius" value="0.08"/>
-  <xacro:property name="wheel_width" value="0.04"/>
+  <xacro:property name="chassis_length" value="0.8"/>
+  <xacro:property name="chassis_width"  value="0.8"/>
+  <xacro:property name="chassis_height" value="0.6"/>
+  <xacro:property name="wheel_radius"   value="0.08"/>
+  <xacro:property name="wheel_width"    value="0.08"/>
   <xacro:property name="wheel_x" value="0.15"/>
   <xacro:property name="wheel_y" value="0.21"/>
   <xacro:property name="chassis_mass" value="20.0"/>
   <xacro:property name="wheel_mass" value="1.2"/>
-  <xacro:property name="caster_mass" value="0.5"/>
   <link name="base_footprint"/>
   <link name="base_link">
@@ -18,12 +17,12 @@
       <inertia ixx="0.433" ixy="0.0" ixz="0.0" iyy="0.563" iyz="0.0" izz="0.683"/>
     </inertial>
+    <!-- OBJ from Blender in metres; scale = 1 1 1. MTL auto-loaded by matching base name. -->
+    <!-- xyz offsets the mesh so its geometric centre aligns with the base_link frame origin. -->
     <visual>
-      <origin xyz="0 0 ${chassis_height/2.0}" rpy="0 0 0"/>
+      <origin xyz="0.9 0 0.06" rpy="1.5708 0 0"/>
       <geometry>
-        <box size="${chassis_length} ${chassis_width} ${chassis_height}"/>
+        <mesh filename="package://anhc_description/meshes/anhc_botrl/visual/obj/baselink.obj"
+              scale="1 1 1"/>
       </geometry>
-      <material name="dark_gray">
-        <color rgba="0.25 0.25 0.28 1.0"/>
-      </material>
     </visual>
     <collision>
@@ -39,5 +38,8 @@
     <origin xyz="0 0 0" rpy="0 0 0"/>
   </joint>
-  <xacro:macro name="wheel_link" params="name x y">
+  <!-- mesh_file: OBJ filename under meshes/anhc_botrl/visual/obj/ -->
+  <!-- vis_x/y/z: visual origin offset in link frame (forward / left-right / up-down).       -->
+  <!-- vis_rpy:   visual rotation; default +90° roll. Use -1.5708 0 0 to flip inner/outer.  -->
+  <xacro:macro name="wheel_link" params="name x y mesh_file vis_x vis_y vis_z vis_rpy:='1.5708 0 0'">
     <link name="${name}">
       <inertial>
@@ -46,12 +48,11 @@
         <inertia ixx="0.0022" ixy="0.0" ixz="0.0" iyy="0.0040" iyz="0.0" izz="0.0022"/>
       </inertial>
+      <!-- OBJ from Blender in metres; scale = 1 1 1. MTL auto-loaded by matching base name. -->
       <visual>
-        <origin xyz="0 0 0" rpy="1.5708 0 0"/>
+        <origin xyz="${vis_x} ${vis_y} ${vis_z}" rpy="${vis_rpy}"/>
         <geometry>
-          <cylinder radius="${wheel_radius}" length="${wheel_width}"/>
+          <mesh filename="package://anhc_description/meshes/anhc_botrl/visual/obj/${mesh_file}"
+                scale="1 1 1"/>
         </geometry>
-        <material name="black">
-          <color rgba="0.05 0.05 0.05 1.0"/>
-        </material>
       </visual>
       <collision>
@@ -71,32 +72,13 @@
     </joint>
   </xacro:macro>
-  <xacro:wheel_link name="left_wheel" x="${wheel_x}" y="${wheel_y}"/>
-  <xacro:wheel_link name="right_wheel" x="${wheel_x}" y="-${wheel_y}"/>
-  <xacro:macro name="caster_wheel" params="name x y">
-    <link name="${name}">
-      <inertial>
-        <origin xyz="0 0 0" rpy="0 0 0"/>
-        <mass value="${caster_mass}"/>
-        <inertia ixx="0.0007" ixy="0.0" ixz="0.0" iyy="0.0009" iyz="0.0" izz="0.0007"/>
-      </inertial>
-      <visual>
-        <origin xyz="0 0 0" rpy="1.5708 0 0"/>
-        <geometry>
-          <sphere radius="0.04"/>
-        </geometry>
-        <material name="silver">
-          <color rgba="0.7 0.7 0.75 1.0"/>
-        </material>
-      </visual>
-      <!-- No collision: passive casters + Gazebo contact solver often inject yaw torque. -->
-    </link>
-    <joint name="${name}_joint" type="fixed">
-      <parent link="base_link"/>
-      <child link="${name}"/>
-      <origin xyz="${x} ${y} 0.04" rpy="0 0 0"/>
-    </joint>
-  </xacro:macro>
-  <xacro:caster_wheel name="rear_left_caster" x="-0.18" y="0.16"/>
-  <xacro:caster_wheel name="rear_right_caster" x="-0.18" y="-0.16"/>
+  <!-- Front wheels (powered, drive wheels) -->
+  <xacro:wheel_link name="front_left_wheel"  x="${wheel_x}"                    y="${wheel_y}"  mesh_file="front_left_wheel.obj"  vis_x="-0.0085" vis_y="0.0781"  vis_z="-0.0921"/>
+  <!-- vis_y/z computed for exact mirror symmetry with front_left (center_y=-0.05, center_z=-0.02) -->
+  <xacro:wheel_link name="front_right_wheel" x="${wheel_x}"                    y="-${wheel_y}" mesh_file="back_right_wheel.obj"  vis_x="-0.22" vis_y="0.1964"  vis_z="0.0542"  vis_rpy="-1.5708 0 0"/>
+  <!-- Rear wheels — same joint type (continuous), driven passively via physics -->
+  <!-- back_left: vis_x +0.04 (≈ half wheel width forward) -->
+  <xacro:wheel_link name="back_left_wheel"   x="-${chassis_length/2.0 - 0.05}" y="${wheel_y}"  mesh_file="back_left_wheel.obj"   vis_x="0.12"    vis_y="0.0655"  vis_z="-0.0986"/>
+  <!-- vis_y/z computed for exact mirror symmetry with back_left (center_y=-0.05, center_z=-0.021) -->
+  <xacro:wheel_link name="back_right_wheel"  x="-${chassis_length/2.0 - 0.05}" y="-${wheel_y}" mesh_file="front_right_wheel.obj" vis_x="0.50"    vis_y="0.0234"  vis_z="-0.0782"/>
   <link name="lidar_link">
     <inertial>
@@ -105,8 +87,11 @@
       <inertia ixx="0.0004" ixy="0.0" ixz="0.0" iyy="0.0004" iyz="0.0" izz="0.0005"/>
     </inertial>
+    <!-- OBJ from Blender in metres; scale = 1 1 1. MTL auto-loaded by matching base name. -->
     <visual>
-      <origin xyz="0 0 0" rpy="0 0 0"/>
-      <geometry><cylinder radius="0.04" length="0.05"/></geometry>
-      <material name="blue"><color rgba="0.2 0.2 0.9 1.0"/></material>
+      <origin xyz="0.0132 0.0205 0.0000" rpy="1.5708 0 3.14159"/>
+      <geometry>
+        <mesh filename="package://anhc_description/meshes/anhc_botrl/visual/obj/lidar.obj"
+              scale="1 1 1"/>
+      </geometry>
     </visual>
     <!-- No collision: avoid spurious contacts with world mesh; lidar is not physical. -->
@@ -115,5 +100,5 @@
     <parent link="base_link"/>
     <child link="lidar_link"/>
-    <origin xyz="0 0 0.30" rpy="0 0 0"/>
+    <origin xyz="0.1 0 0.4" rpy="0 0 0"/>
   </joint>
   <link name="camera_link">
@@ -123,8 +108,11 @@
       <inertia ixx="0.0009" ixy="0.0" ixz="0.0" iyy="0.0010" iyz="0.0" izz="0.0008"/>
     </inertial>
+    <!-- OBJ from Blender in metres; scale = 1 1 1. MTL auto-loaded by matching base name. -->
     <visual>
-      <origin xyz="0 0 0" rpy="0 0 0"/>
-      <geometry><box size="0.08 0.06 0.05"/></geometry>
-      <material name="navy"><color rgba="0.1 0.1 0.5 1.0"/></material>
+      <origin xyz="0.0133 0.0128 0.0000" rpy="1.5708 0 0"/>
+      <geometry>
+        <mesh filename="package://anhc_description/meshes/anhc_botrl/visual/obj/camera.obj"
+              scale="1 1 1"/>
+      </geometry>
     </visual>
     <collision>
@@ -136,5 +124,5 @@
     <parent link="base_link"/>
     <child link="camera_link"/>
-    <origin xyz="0.22 0 0.20" rpy="0 0.1745 0"/>
+    <origin xyz="0.22 0 0.7" rpy="0 0 0"/>
   </joint>
   <link name="imu_link">

Commit message: [Sim] - migrate office_v2 map flow and rebuild wheel setup
Switch office_v2 navigation to SLAM-first flow and migrate the world mesh to OBJ/MTL with stable rendering defaults. Replace custom wheel OBJ dependencies with primitive wheels and robust joint-state publishing so RViz wheel TF remains available.

Made-with: Cursor

File: src/anhc_description/urdf/anhc_bot.gazebo.xacro (robot description, xacro)
@@ -78,4 +78,12 @@
   </gazebo>
   <gazebo>
+    <plugin filename="gz-sim-joint-state-publisher-system" name="gz::sim::systems::JointStatePublisher">
+      <joint_name>front_left_wheel_joint</joint_name>
+      <joint_name>front_right_wheel_joint</joint_name>
+      <joint_name>back_left_wheel_joint</joint_name>
+      <joint_name>back_right_wheel_joint</joint_name>
+    </plugin>
+  </gazebo>
+  <gazebo>
     <plugin filename="gz-sim-diff-drive-system" name="gz::sim::systems::DiffDrive">
       <!-- 4WD: both left wheels share the same velocity command, same for right -->

File: src/anhc_description/urdf/anhc_bot.urdf.xacro (robot description, xacro)
@@ -38,8 +38,6 @@
     <origin xyz="0 0 0" rpy="0 0 0"/>
   </joint>
-  <!-- mesh_file: OBJ filename under meshes/anhc_botrl/visual/obj/ -->
-  <!-- vis_x/y/z: visual origin offset in link frame (forward / left-right / up-down).       -->
-  <!-- vis_rpy:   visual rotation; default +90° roll. Use -1.5708 0 0 to flip inner/outer.  -->
-  <xacro:macro name="wheel_link" params="name x y mesh_file vis_x vis_y vis_z vis_rpy:='1.5708 0 0'">
+  <!-- Primitive wheel model (no external OBJ dependency). -->
+  <xacro:macro name="wheel_link" params="name x y">
     <link name="${name}">
       <inertial>
@@ -48,11 +46,12 @@
         <inertia ixx="0.0022" ixy="0.0" ixz="0.0" iyy="0.0040" iyz="0.0" izz="0.0022"/>
       </inertial>
-      <!-- OBJ from Blender in metres; scale = 1 1 1. MTL auto-loaded by matching base name. -->
       <visual>
-        <origin xyz="${vis_x} ${vis_y} ${vis_z}" rpy="${vis_rpy}"/>
+        <origin xyz="0 0 0" rpy="1.5708 0 0"/>
         <geometry>
-          <mesh filename="package://anhc_description/meshes/anhc_botrl/visual/obj/${mesh_file}"
-                scale="1 1 1"/>
+          <cylinder radius="${wheel_radius}" length="${wheel_width}"/>
         </geometry>
+        <material name="wheel_dark_gray">
+          <color rgba="0.10 0.10 0.10 1.0"/>
+        </material>
       </visual>
       <collision>
@@ -73,12 +72,9 @@
   </xacro:macro>
   <!-- Front wheels (powered, drive wheels) -->
-  <xacro:wheel_link name="front_left_wheel"  x="${wheel_x}"                    y="${wheel_y}"  mesh_file="front_left_wheel.obj"  vis_x="-0.0085" vis_y="0.0781"  vis_z="-0.0921"/>
-  <!-- vis_y/z computed for exact mirror symmetry with front_left (center_y=-0.05, center_z=-0.02) -->
-  <xacro:wheel_link name="front_right_wheel" x="${wheel_x}"                    y="-${wheel_y}" mesh_file="back_right_wheel.obj"  vis_x="-0.22" vis_y="0.1964"  vis_z="0.0542"  vis_rpy="-1.5708 0 0"/>
+  <xacro:wheel_link name="front_left_wheel"  x="${wheel_x}"                    y="${wheel_y}"/>
+  <xacro:wheel_link name="front_right_wheel" x="${wheel_x}"                    y="-${wheel_y}"/>
   <!-- Rear wheels — same joint type (continuous), driven passively via physics -->
-  <!-- back_left: vis_x +0.04 (≈ half wheel width forward) -->
-  <xacro:wheel_link name="back_left_wheel"   x="-${chassis_length/2.0 - 0.05}" y="${wheel_y}"  mesh_file="back_left_wheel.obj"   vis_x="0.12"    vis_y="0.0655"  vis_z="-0.0986"/>
-  <!-- vis_y/z computed for exact mirror symmetry with back_left (center_y=-0.05, center_z=-0.021) -->
-  <xacro:wheel_link name="back_right_wheel"  x="-${chassis_length/2.0 - 0.05}" y="-${wheel_y}" mesh_file="front_right_wheel.obj" vis_x="0.50"    vis_y="0.0234"  vis_z="-0.0782"/>
+  <xacro:wheel_link name="back_left_wheel"   x="-${chassis_length/2.0 - 0.05}" y="${wheel_y}"/>
+  <xacro:wheel_link name="back_right_wheel"  x="-${chassis_length/2.0 - 0.05}" y="-${wheel_y}"/>
   <link name="lidar_link">
     <inertial>
